File: oya45.sch (KiCad schematic (older format))
At the start: 24 parts, among them SW1 SW_Push, U1 ATmega32U4-AU, Y1 Crystal_GND24_Small

Commit message: schematics finish
Parts:
- C1, C2, C3, C4, C5, C6, C7: footprint (none) -> Capacitor_SMD:C_0805_2012Metric
- D1, D2, D3, D4: footprint (none) -> Diode_SMD:D_SOD-123
- F1: footprint (none) -> Fuse:Fuse_1206_3216Metric
- MX1, MX2, MX3, MX4: footprint (none) -> MX_Only:MXOnly-1U-NoLED
- R1, R2, R3, R4: footprint (none) -> Resistor_SMD:R_0805_2012Metric
- SW1: footprint (none) -> random-keyboard-parts:SKQG-1155865
- USB1: footprint (none) -> random-keyboard-parts:Molex-0548190589
- Y1: footprint (none) -> Crystal:Crystal_SMD_3225-4Pin_3.2x2.5mm
Changed lines of the file:
@@
 EESchema Schematic File Version 4
+LIBS:oya45-cache
 EELAYER 30 0
 EELAYER END
@@
 F 0 "R4" V 3704 3950 50  0000 C CNN
 F 1 "10k" V 3795 3950 50  0000 C CNN
-F 2 "" H 3900 3950 50  0001 C CNN
+F 2 "Resistor_SMD:R_0805_2012Metric" H 3900 3950 50  0001 C CNN
 F 3 "~" H 3900 3950 50  0001 C CNN
 	1    3900 3950
@@
 F 0 "R2" V 1304 2850 50  0000 C CNN
 F 1 "22" V 1395 2850 50  0000 C CNN
-F 2 "" H 1500 2850 50  0001 C CNN
+F 2 "Resistor_SMD:R_0805_2012Metric" H 1500 2850 50  0001 C CNN
 F 3 "~" H 1500 2850 50  0001 C CNN
 	1    1500 2850
@@
 F 0 "R1" V 954 2950 50  0000 C CNN
 F 1 "22" V 1045 2950 50  0000 C CNN
-F 2 "" H 1150 2950 50  0001 C CNN
+F 2 "Resistor_SMD:R_0805_2012Metric" H 1150 2950 50  0001 C CNN
 F 3 "~" H 1150 2950 50  0001 C CNN
 	1    1150 2950
@@
 F 0 "C6" H 1542 3296 50  0000 L CNN
 F 1 "1uF" H 1542 3205 50  0000 L CNN
-F 2 "" H 1450 3250 50  0001 C CNN
+F 2 "Capacitor_SMD:C_0805_2012Metric" H 1450 3250 50  0001 C CNN
 F 3 "~" H 1450 3250 50  0001 C CNN
 	1    1450 3250
@@
 F 0 "C1" H 892 4196 50  0000 L CNN
 F 1 "0.1uF" H 892 4105 50  0000 L CNN
-F 2 "" H 800 4150 50  0001 C CNN
+F 2 "Capacitor_SMD:C_0805_2012Metric" H 800 4150 50  0001 C CNN
 F 3 "~" H 800 4150 50  0001 C CNN
 	1    800  4150
@@
 F 0 "C4" H 1142 4196 50  0000 L CNN
 F 1 "0.1uF" H 1142 4105 50  0000 L CNN
-F 2 "" H 1050 4150 50  0001 C CNN
+F 2 "Capacitor_SMD:C_0805_2012Metric" H 1050 4150 50  0001 C CNN
 F 3 "~" H 1050 4150 50  0001 C CNN
 	1    1050 4150
@@
 F 0 "C5" H 1392 4196 50  0000 L CNN
 F 1 "0.1uF" H 1392 4105 50  0000 L CNN
-F 2 "" H 1300 4150 50  0001 C CNN
+F 2 "Capacitor_SMD:C_0805_2012Metric" H 1300 4150 50  0001 C CNN
 F 3 "~" H 1300 4150 50  0001 C CNN
 	1    1300 4150
@@
 F 0 "C7" H 1642 4196 50  0000 L CNN
 F 1 "0.1uF" H 1642 4105 50  0000 L CNN
-F 2 "" H 1550 4150 50  0001 C CNN
+F 2 "Capacitor_SMD:C_0805_2012Metric" H 1550 4150 50  0001 C CNN
 F 3 "~" H 1550 4150 50  0001 C CNN
 	1    1550 4150
@@
 F 0 "Y1" V 1304 2294 50  0000 L CNN
 F 1 "Crystal_GND24_Small" V 1395 2294 50  0000 L CNN
-F 2 "" H 1350 2150 50  0001 C CNN
+F 2 "Crystal:Crystal_SMD_3225-4Pin_3.2x2.5mm" H 1350 2150 50  0001 C CNN
 F 3 "~" H 1350 2150 50  0001 C CNN
 	1    1350 2150
@@
 F 0 "C2" V 721 2000 50  0000 C CNN
 F 1 "22pF" V 812 2000 50  0000 C CNN
-F 2 "" H 950 2000 50  0001 C CNN
+F 2 "Capacitor_SMD:C_0805_2012Metric" H 950 2000 50  0001 C CNN
 F 3 "~" H 950 2000 50  0001 C CNN
 	1    950  2000
@@
 F 0 "C3" V 721 2300 50  0000 C CNN
 F 1 "22pF" V 812 2300 50  0000 C CNN
-F 2 "" H 950 2300 50  0001 C CNN
+F 2 "Capacitor_SMD:C_0805_2012Metric" H 950 2300 50  0001 C CNN
 F 3 "~" H 950 2300 50  0001 C CNN
 	1    950  2300
@@
 F 0 "SW1" H 1600 2135 50  0000 C CNN
 F 1 "SW_Push" H 1600 2044 50  0000 C CNN
-F 2 "" H 1600 2050 50  0001 C CNN
+F 2 "random-keyboard-parts:SKQG-1155865" H 1600 2050 50  0001 C CNN
 F 3 "~" H 1600 2050 50  0001 C CNN
 	1    1600 1850
@@
 F 0 "R3" H 1909 1496 50  0000 L CNN
 F 1 "10k" H 1909 1405 50  0000 L CNN
-F 2 "" H 1850 1450 50  0001 C CNN
+F 2 "Resistor_SMD:R_0805_2012Metric" H 1850 1450 50  0001 C CNN
 F 3 "~" H 1850 1450 50  0001 C CNN
 	1    1850 1450
@@
 F 0 "USB1" V 5037 1817 60  0000 C CNN
 F 1 "Molex-0548190589" V 4931 1817 60  0000 C CNN
-F 2 "" H 4500 1850 60  0001 C CNN
+F 2 "random-keyboard-parts:Molex-0548190589" H 4500 1850 60  0001 C CNN
 F 3 "" H 4500 1850 60  0001 C CNN
 	1    4500 1850
@@
 F 0 "F1" V 5695 1650 50  0000 C CNN
 F 1 "500mA" V 5786 1650 50  0000 C CNN
-F 2 "" H 5950 1450 50  0001 L CNN
+F 2 "Fuse:Fuse_1206_3216Metric" H 5950 1450 50  0001 L CNN
 F 3 "~" H 5900 1650 50  0001 C CNN
 	1    5900 1650
@@
 F 0 "MX1" H 6483 3073 60  0000 C CNN
 F 1 "MX-NoLED" H 6483 2999 20  0000 C CNN
-F 2 "" H 5825 2825 60  0001 C CNN
+F 2 "MX_Only:MXOnly-1U-NoLED" H 5825 2825 60  0001 C CNN
 F 3 "" H 5825 2825 60  0001 C CNN
 	1    6450 2850
@@
 F 0 "D1" V 6346 3032 50  0000 R CNN
 F 1 "SOD_123" V 6255 3032 50  0000 R CNN
-F 2 "" V 6300 3100 50  0001 C CNN
+F 2 "Diode_SMD:D_SOD-123" V 6300 3100 50  0001 C CNN
 F 3 "~" V 6300 3100 50  0001 C CNN
 	1    6300 3100
@@
 F 0 "MX3" H 7083 3073 60  0000 C CNN
 F 1 "MX-NoLED" H 7083 2999 20  0000 C CNN
-F 2 "" H 6425 2825 60  0001 C CNN
+F 2 "MX_Only:MXOnly-1U-NoLED" H 6425 2825 60  0001 C CNN
 F 3 "" H 6425 2825 60  0001 C CNN
 	1    7050 2850
@@
 F 0 "MX4" H 7083 3723 60  0000 C CNN
 F 1 "MX-NoLED" H 7083 3649 20  0000 C CNN
-F 2 "" H 6425 3475 60  0001 C CNN
+F 2 "MX_Only:MXOnly-1U-NoLED" H 6425 3475 60  0001 C CNN
 F 3 "" H 6425 3475 60  0001 C CNN
 	1    7050 3500
@@
 F 0 "MX2" H 6483 3723 60  0000 C CNN
 F 1 "MX-NoLED" H 6483 3649 20  0000 C CNN
-F 2 "" H 5825 3475 60  0001 C CNN
+F 2 "MX_Only:MXOnly-1U-NoLED" H 5825 3475 60  0001 C CNN
 F 3 "" H 5825 3475 60  0001 C CNN
 	1    6450 3500
@@
 F 0 "D3" V 6946 3032 50  0000 R CNN
 F 1 "SOD_123" V 6855 3032 50  0000 R CNN
-F 2 "" V 6900 3100 50  0001 C CNN
+F 2 "Diode_SMD:D_SOD-123" V 6900 3100 50  0001 C CNN
 F 3 "~" V 6900 3100 50  0001 C CNN
 	1    6900 3100
@@
 F 0 "D4" V 6946 3682 50  0000 R CNN
 F 1 "SOD_123" V 6855 3682 50  0000 R CNN
-F 2 "" V 6900 3750 50  0001 C CNN
+F 2 "Diode_SMD:D_SOD-123" V 6900 3750 50  0001 C CNN
 F 3 "~" V 6900 3750 50  0001 C CNN
 	1    6900 3750
@@
 F 0 "D2" V 6346 3682 50  0000 R CNN
 F 1 "SOD_123" V 6255 3682 50  0000 R CNN
-F 2 "" V 6300 3750 50  0001 C CNN
+F 2 "Diode_SMD:D_SOD-123" V 6300 3750 50  0001 C CNN
 F 3 "~" V 6300 3750 50  0001 C CNN
 	1    6300 3750

Commit message: schematicfinish1
Parts:
- C7: value 0.1uF -> 10uF
- Y1: value Crystal_GND24_Small -> 16MHz
Changed lines of the file:
@@
-$EndComp
-$Comp
-L Device:C_Small C7
-U 1 1 612C17BD
-P 1550 4150
-F 0 "C7" H 1642 4196 50  0000 L CNN
-F 1 "0.1uF" H 1642 4105 50  0000 L CNN
-F 2 "Capacitor_SMD:C_0805_2012Metric" H 1550 4150 50  0001 C CNN
-F 3 "~" H 1550 4150 50  0001 C CNN
-	1    1550 4150
-	1    0    0    -1
 $EndComp
 $Comp
@@
 P 1350 2150
 F 0 "Y1" V 1304 2294 50  0000 L CNN
-F 1 "Crystal_GND24_Small" V 1395 2294 50  0000 L CNN
+F 1 "16MHz" V 1395 2294 50  0000 L CNN
 F 2 "Crystal:Crystal_SMD_3225-4Pin_3.2x2.5mm" H 1350 2150 50  0001 C CNN
 F 3 "~" H 1350 2150 50  0001 C CNN
@@
 Text GLabel 5950 3850 0    50   Input ~ 0
 ROW1
+$Comp
+L Device:C_Small C7
+U 1 1 612C17BD
+P 1550 4150
+F 0 "C7" H 1642 4196 50  0000 L CNN
+F 1 "10uF" H 1642 4105 50  0000 L CNN
+F 2 "Capacitor_SMD:C_0805_2012Metric" H 1550 4150 50  0001 C CNN
+F 3 "~" H 1550 4150 50  0001 C CNN
+	1    1550 4150
+	1    0    0    -1
+$EndComp
 $EndSCHEMATC
