File: oya45.kicad_pcb (KiCad board)
At the start: 2 copper layers, 24 parts, among them SW1 SW_Push, U1 ATmega32U4-AU, Y1 Crystal_GND24_Small

Commit message: test finish
Parts:
- C1, C4, C5, C6, F1, R1, R2, R3, R4, SW1, USB1: moved to B.Cu
- C7: value 0.1uF -> 10uF; moved to B.Cu
- Y1: value Crystal_GND24_Small -> 16MHz
- moved C5 52.8 mm to (149.2, 113.5), turned to 180 degrees
- moved R4 52.1 mm to (155.6, 108.0), turned to 90 degrees
- moved C7 43.7 mm to (141.3, 113.5)
- moved C1 43.0 mm to (155.6, 100.0), turned to 90 degrees
- moved C6 31.8 mm to (133.3, 102.4), turned to 270 degrees
- moved SW1 30.6 mm to (122.2, 104.0), turned to 270 degrees
- moved C4 25.7 mm to (134.9, 96.0), turned to 90 degrees
- moved R1 24.5 mm to (120.7, 90.5), turned to 90 degrees
- moved R3 23.3 mm to (131.8, 96.0), turned to 90 degrees
- moved F1 23.1 mm to (120.7, 96.0), turned to 90 degrees
- moved R2 14.2 mm to (123.8, 90.5), turned to 90 degrees
- moved USB1 13.4 mm to (122.2, 81.0), turned to 270 degrees
- moved C2 6.55 mm to (149.2, 92.9)
- moved C3 6.55 mm to (139.7, 92.9)
- moved U1 6.55 mm to (145.3, 103.2)
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Routing:
- net GND: track 0.00 -> 35.0 mm
- net Net-(R1-Pad1): track 0.00 -> 29.5 mm
- net Net-(R2-Pad1): track 0.00 -> 25.4 mm
- net Net-(C3-Pad1): track 0.00 -> 11.9 mm
- net +5V: track 0.00 -> 9.20 mm
- net Net-(C2-Pad1): track 0.00 -> 7.59 mm
- net D-: track 0.00 -> 5.07 mm
- net D+: track 0.00 -> 4.83 mm
Other:
- net class Default: trace_width 0.25 -> 0.254
- net class power added: clearance 0.2, trace_width 0.381, via_dia 0.8, via_drill 0.4

Commit message: Add submodules
Routing:
- net Net-(D3-Pad2): track 0.00 -> 7.23 mm
- net +5V: track 9.20 -> 14.2 mm
Changed lines of the file:
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@@
     (thickness 1.6)
     (drawings 2)
-    (tracks 53)
+    (tracks 58)
     (zones 0)
     (modules 24)
@@
   (segment (start 135.571751 96.346999) (end 142.643651 96.346999) (width 0.381) (layer B.Cu) (net 2))
   (segment (start 134.9375 96.98125) (end 135.571751 96.346999) (width 0.381) (layer B.Cu) (net 2))
+  (segment (start 141.25625 112.6) (end 140.35 113.50625) (width 0.381) (layer B.Cu) (net 2))
+  (segment (start 141.25625 108.8875) (end 141.25625 112.6) (width 0.381) (layer B.Cu) (net 2))
   (segment (start 145.25625 96.4835) (end 145.25625 97.4875) (width 0.254) (layer B.Cu) (net 3))
   (segment (start 145.25625 94.879) (end 145.25625 96.4835) (width 0.254) (layer B.Cu) (net 3))
@@
   (segment (start 144.45625 95.24375) (end 144.45625 97.4875) (width 0.254) (layer B.Cu) (net 4))
   (segment (start 143.858251 94.645751) (end 144.45625 95.24375) (width 0.254) (layer B.Cu) (net 4))
+  (segment (start 176.2125 105.596) (end 176.2125 106.3) (width 0.254) (layer B.Cu) (net 10))
+  (segment (start 173.4865 102.87) (end 176.2125 105.596) (width 0.254) (layer B.Cu) (net 10))
+  (segment (start 170.815 102.87) (end 173.4865 102.87) (width 0.254) (layer B.Cu) (net 10))
   (segment (start 121.4375 88.10625) (end 120.65 88.89375) (width 0.254) (layer B.Cu) (net 15))
   (segment (start 121.4375 84.80625) (end 121.4375 88.10625) (width 0.254) (layer B.Cu) (net 15))
